Commit message: mapping works

File: urdf/robot.xacro (robot description, xacro)
@@ -16,10 +16,10 @@
     <link name="base_footprint"></link>
     <joint name="base_footprint_joint" type="fixed">
-        <origin xyz="0 0 -${wr}" rpy="0 0 0"/>
+        <origin xyz="0 0 0" rpy="0 0 0"/>
         <parent link="base_link"/>
         <child link="base_footprint"/>
     </joint>
     <joint name="chassis_joint" type="fixed">
-		<origin xyz="0 0 0" rpy="0 0 0" />
+		<origin xyz="0 0 ${wr}" rpy="0 0 0" />
         <parent link="base_link"/>
         <child link="chassis" />
@@ -97,4 +97,10 @@
         <origin xyz="0.25 0 0.05" rpy="0 0 0"/>
     </joint>
+	<link name="camera_optical"/>
+	<joint name="camera_optical_joint" type="fixed">
+		<origin xyz="0 0 0" rpy="${-pi/2} 0 ${-pi/2}"/>
+        <parent link="camera"/>
+        <child link="camera_optical"/>
+	</joint>
     <link name="laser">
         <inertial>
@@ -116,5 +122,5 @@
         <parent link="chassis"/>
         <child link="laser"/>
-        <origin xyz="0.0 0 0.1" rpy="0 0 0"/>
+        <origin xyz="0.0 0 0.11" rpy="0 0 0"/>
     </joint>
 </robot>

Commit message: add figures

File: urdf/robot.xacro (robot description, xacro)
@@ -95,5 +95,5 @@
         <parent link="chassis"/>
         <child link="camera"/>
-        <origin xyz="0.25 0 0.05" rpy="0 0 0"/>
+		<origin xyz="0.25 0 0.2" rpy="0 ${10*deg} 0"/>
     </joint>
 	<link name="camera_optical"/>

Commit message: add custom configuration + now supports localization

File: urdf/robot.xacro (robot description, xacro)
@@ -46,5 +46,5 @@
 			<origin xyz="-0.15 0 ${-wr+cr}" rpy=" 0 0 0"/>
             <geometry>
-				<sphere radius="${cr}"/>
+				<sphere radius="${cr*0.99}"/>
             </geometry>
         </collision>
@@ -58,5 +58,5 @@
 			<origin xyz="0.15 0 ${-wr+cr}" rpy=" 0 0 0"/>
             <geometry>
-				<sphere radius="${cr}"/>
+				<sphere radius="${cr*0.99}"/>
             </geometry>
         </collision>
